File: SpacePort.kicad_pcb (KiCad board)
At the start: 2 copper layers, 11.2 x 19.6 mm, 23 parts, among them U1 AP2112K-3.3

Commit message: knew i'd forget something. now includes the parts lib. also fixed the linking
Parts:
- C1, C8: footprint modchip-2layer:0805-NO -> SpacePort:0805-NO
- C3, C4: footprint modchip-2layer:0603-NO -> SpacePort:0603-NO
- TP1, TP11, TP12, TP13, TP14, TP15, TP16, TP17: footprint modchip-2layer:PAD.03X.03 -> SpacePort:PAD.03X.03
- TP2, TP3, TP4, TP5, TP6, TP7, TP8, TP9: footprint modchip-2layer:TP20SQ -> SpacePort:TP20SQ
- U$1: footprint modchip-2layer:32-TQFP -> SpacePort:32-TQFP
- U$3: footprint modchip-2layer:APA102_2020 -> SpacePort:APA102_2020
- U1: footprint modchip-2layer:SOT23-5 -> SpacePort:SOT23-5
Changed lines of the file:
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@@
     (add_net VBAT)
   )
-  (module modchip-2layer:0805-NO (layer Top)
+  (module SpacePort:0805-NO (layer Top)
     (at 144.3736 110.1697 270)
     (fp_text reference C8 (at 2.032 0.127 270) (layer F.SilkS) hide
@@
       (net 2 3.3V) (solder_mask_margin 0.1397))
   )
-  (module modchip-2layer:0805-NO (layer Top)
+  (module SpacePort:0805-NO (layer Top)
     (at 150.4696 110.1217 90)
     (fp_text reference C1 (at 2.032 0.127 90) (layer F.SilkS) hide
@@
       (net 3 VBAT) (solder_mask_margin 0.1397))
   )
-  (module modchip-2layer:SOT23-5 (layer Top)
+  (module SpacePort:SOT23-5 (layer Top)
     (at 147.4071 110.0737 90)
     (descr "<b>Small Outline Transistor</b> - 5 Pin")
@@
       (net 3 VBAT) (solder_mask_margin 0.1397))
   )
-  (module modchip-2layer:0603-NO (layer Top)
+  (module SpacePort:0603-NO (layer Top)
     (at 149.3901 98.2472)
     (fp_text reference C3 (at 1.778 0.127) (layer F.SilkS) hide
@@
       (net 5 "Net-(C3-Pad1)") (solder_mask_margin 0.1397))
   )
-  (module modchip-2layer:32-TQFP (layer Top)
+  (module SpacePort:32-TQFP (layer Top)
     (at 149.0726 103.4542)
     (fp_text reference U$1 (at 0 0) (layer F.SilkS) hide
@@
       (net 31 "Net-(TP13-PadP$1)") (solder_mask_margin 0.1397))
   )
-  (module modchip-2layer:TP20SQ (layer Top)
+  (module SpacePort:TP20SQ (layer Top)
     (at 152.6921 113.4237)
     (descr "<b>TEST PAD</b>")
@@
       (net 1 GND) (solder_mask_margin 0.1397))
   )
-  (module modchip-2layer:TP20SQ (layer Top)
+  (module SpacePort:TP20SQ (layer Top)
     (at 152.5651 109.4867)
     (descr "<b>TEST PAD</b>")
@@
       (net 3 VBAT) (solder_mask_margin 0.1397))
   )
-  (module modchip-2layer:TP20SQ (layer Top)
+  (module SpacePort:TP20SQ (layer Top)
     (at 149.9743 96.4819)
     (descr "<b>TEST PAD</b>")
@@
       (net 11 /D+) (solder_mask_margin 0.1397))
   )
-  (module modchip-2layer:TP20SQ (layer Top)
+  (module SpacePort:TP20SQ (layer Top)
     (at 147.1803 96.4819)
     (descr "<b>TEST PAD</b>")
@@
       (net 12 /D-) (solder_mask_margin 0.1397))
   )
-  (module modchip-2layer:TP20SQ (layer Top)
+  (module SpacePort:TP20SQ (layer Top)
     (at 144.3101 113.4237)
     (descr "<b>TEST PAD</b>")
@@
       (net 6 /SWD) (solder_mask_margin 0.1397))
   )
-  (module modchip-2layer:TP20SQ (layer Top)
+  (module SpacePort:TP20SQ (layer Top)
     (at 147.1041 113.4237)
     (descr "<b>TEST PAD</b>")
@@
       (net 7 /SWC) (solder_mask_margin 0.1397))
   )
-  (module modchip-2layer:TP20SQ (layer Top)
+  (module SpacePort:TP20SQ (layer Top)
     (at 149.8981 113.4237)
     (descr "<b>TEST PAD</b>")
@@
       (net 2 3.3V) (solder_mask_margin 0.1397))
   )
-  (module modchip-2layer:TP20SQ (layer Top)
+  (module SpacePort:TP20SQ (layer Top)
     (at 152.7683 96.4819)
     (descr "<b>TEST PAD</b>")
@@
       (net 9 /RST) (solder_mask_margin 0.1397))
   )
-  (module modchip-2layer:PAD.03X.03 (layer Top)
+  (module SpacePort:PAD.03X.03 (layer Top)
     (at 143.8275 100.4189)
     (descr "<h3>Electrically Conductive Pad 0.03\" Circle</h3>\nUsed as a test point connection for pogo pins or other debugging tools. \n<p>Specifications:\n<li>Area: 0.03\" x 0.03\"</li>\n</ul></p>\n<p>Example device(s):\n<ul><li>TEST_POINT</li>\n</ul></p>")
@@
       (net 28 /DI) (solder_mask_margin 0.1397))
   )
-  (module modchip-2layer:PAD.03X.03 (layer Top)
+  (module SpacePort:PAD.03X.03 (layer Top)
     (at 143.8275 101.4349)
     (descr "<h3>Electrically Conductive Pad 0.03\" Circle</h3>\nUsed as a test point connection for pogo pins or other debugging tools. \n<p>Specifications:\n<li>Area: 0.03\" x 0.03\"</li>\n</ul></p>\n<p>Example device(s):\n<ul><li>TEST_POINT</li>\n</ul></p>")
@@
       (net 29 /CI) (solder_mask_margin 0.1397))
   )
-  (module modchip-2layer:PAD.03X.03 (layer Top)
+  (module SpacePort:PAD.03X.03 (layer Top)
     (at 143.8275 102.4001)
     (descr "<h3>Electrically Conductive Pad 0.03\" Circle</h3>\nUsed as a test point connection for pogo pins or other debugging tools. \n<p>Specifications:\n<li>Area: 0.03\" x 0.03\"</li>\n</ul></p>\n<p>Example device(s):\n<ul><li>TEST_POINT</li>\n</ul></p>")
@@
       (net 30 "Net-(TP12-PadP$1)") (solder_mask_margin 0.1397))
   )
-  (module modchip-2layer:PAD.03X.03 (layer Top)
+  (module SpacePort:PAD.03X.03 (layer Top)
     (at 143.8275 103.4161)
     (descr "<h3>Electrically Conductive Pad 0.03\" Circle</h3>\nUsed as a test point connection for pogo pins or other debugging tools. \n<p>Specifications:\n<li>Area: 0.03\" x 0.03\"</li>\n</ul></p>\n<p>Example device(s):\n<ul><li>TEST_POINT</li>\n</ul></p>")
@@
       (net 31 "Net-(TP13-PadP$1)") (solder_mask_margin 0.1397))
   )
-  (module modchip-2layer:PAD.03X.03 (layer Top)
+  (module SpacePort:PAD.03X.03 (layer Top)
     (at 143.8275 104.4829)
     (descr "<h3>Electrically Conductive Pad 0.03\" Circle</h3>\nUsed as a test point connection for pogo pins or other debugging tools. \n<p>Specifications:\n<li>Area: 0.03\" x 0.03\"</li>\n</ul></p>\n<p>Example device(s):\n<ul><li>TEST_POINT</li>\n</ul></p>")
@@
       (net 27 "Net-(TP14-PadP$1)") (solder_mask_margin 0.1397))
   )
-  (module modchip-2layer:PAD.03X.03 (layer Top)
+  (module SpacePort:PAD.03X.03 (layer Top)
     (at 143.8275 105.4989)
     (descr "<h3>Electrically Conductive Pad 0.03\" Circle</h3>\nUsed as a test point connection for pogo pins or other debugging tools. \n<p>Specifications:\n<li>Area: 0.03\" x 0.03\"</li>\n</ul></p>\n<p>Example device(s):\n<ul><li>TEST_POINT</li>\n</ul></p>")
@@
       (net 26 "Net-(TP15-PadP$1)") (solder_mask_margin 0.1397))
   )
-  (module modchip-2layer:PAD.03X.03 (layer Top)
+  (module SpacePort:PAD.03X.03 (layer Top)
     (at 143.8275 106.5149)
     (descr "<h3>Electrically Conductive Pad 0.03\" Circle</h3>\nUsed as a test point connection for pogo pins or other debugging tools. \n<p>Specifications:\n<li>Area: 0.03\" x 0.03\"</li>\n</ul></p>\n<p>Example device(s):\n<ul><li>TEST_POINT</li>\n</ul></p>")
@@
       (net 25 "Net-(TP16-PadP$1)") (solder_mask_margin 0.1397))
   )
-  (module modchip-2layer:PAD.03X.03 (layer Top)
+  (module SpacePort:PAD.03X.03 (layer Top)
     (at 143.8275 107.5309)
     (descr "<h3>Electrically Conductive Pad 0.03\" Circle</h3>\nUsed as a test point connection for pogo pins or other debugging tools. \n<p>Specifications:\n<li>Area: 0.03\" x 0.03\"</li>\n</ul></p>\n<p>Example device(s):\n<ul><li>TEST_POINT</li>\n</ul></p>")
@@
       (net 24 "Net-(TP17-PadP$1)") (solder_mask_margin 0.1397))
   )
-  (module modchip-2layer:APA102_2020 (layer Top)
+  (module SpacePort:APA102_2020 (layer Top)
     (at 145.1991 97.5233 90)
     (fp_text reference U$3 (at 0 0 90) (layer F.SilkS) hide
@@
       (net 28 /DI) (solder_mask_margin 0.1397))
   )
-  (module modchip-2layer:0603-NO (layer Top)
+  (module SpacePort:0603-NO (layer Top)
     (at 145.2753 98.38055 180)
     (fp_text reference C4 (at 1.778 0.127 180) (layer F.SilkS) hide
